File: hardware/Orbital_imager_HiResDev_F1C200s/Orbital_imager_HiResDev_F1C200s.kicad_pcb (KiCad board)
At the start: 2 copper layers, 50 x 50 mm, 26 parts, among them J1 2.54, J2 USB_B, J3 2.54, SW1 SW_SPST, U2 W25Q128, Y1 24MHz

Commit message: ported to C
Parts:
- removed J3: 2.54, Connector_PinHeader_2.54mm:PinHeader_1x12_P2.54mm_Vertical
- added C13: 1uF, Capacitor_SMD:C_0402_1005Metric, F.Cu at (131.0, 72.4)
- added C14: 22nF, Capacitor_SMD:C_0402_1005Metric, F.Cu at (125.4, 60.8)
- added C15: 22uF, Capacitor_SMD:C_0805_2012Metric, F.Cu at (126.2, 62.4)
- added C16: 22uF, Capacitor_SMD:C_0805_2012Metric, F.Cu at (126.2, 64.5)
- added C17: 22uF, Capacitor_SMD:C_0805_2012Metric, F.Cu at (120.1, 57.2)
- added C18: 22uF, Capacitor_SMD:C_0805_2012Metric, F.Cu at (111.3, 68.5)
- added C19: 22nF, Capacitor_SMD:C_0402_1005Metric, F.Cu at (114.9, 63.2)
- added C20: 22uF, Capacitor_SMD:C_0805_2012Metric, F.Cu at (116.5, 62.4)
- added C21: 22uF, Capacitor_SMD:C_0805_2012Metric, F.Cu at (118.6, 62.4)
- added C22: 22uF, Capacitor_SMD:C_0805_2012Metric, F.Cu at (111.3, 79.6)
- added C23: 22nF, Capacitor_SMD:C_0402_1005Metric, F.Cu at (114.9, 74.3)
- added C24: 22uF, Capacitor_SMD:C_0805_2012Metric, F.Cu at (116.5, 73.5)
- added C25: 22uF, Capacitor_SMD:C_0805_2012Metric, F.Cu at (118.6, 73.5)
- added D1: ESD0603, Diode_SMD:D_0603_1608Metric, F.Cu at (133.9, 66.4)
- added D2: GREEN 0603, Diode_SMD:D_0603_1608Metric, F.Cu at (133.9, 68.0)
- added Le1: MPL2520S4R7MHT, Inductor_SMD:L_1008_2520Metric, F.Cu at (123.0, 62.3)
- added Le2: MPL2520S4R7MHT, Inductor_SMD:L_1008_2520Metric, F.Cu at (116.4, 65.6)
- added Le3: MPL2520S4R7MHT, Inductor_SMD:L_1008_2520Metric, F.Cu at (116.4, 76.7)
- added R10: 10k, Resistor_SMD:R_0402_1005Metric, F.Cu at (112.1, 78.0)
- added R11: 100k, Resistor_SMD:R_0402_1005Metric, F.Cu at (112.4, 71.7)
- added R12: 33k, Resistor_SMD:R_0402_1005Metric, F.Cu at (112.4, 72.7)
- added R13: 10k, Resistor_SMD:R_0402_1005Metric, F.Cu at (131.3, 68.0)
- added R4: 68k, Resistor_SMD:R_0402_1005Metric, F.Cu at (128.0, 58.3)
- added R5: 15k, Resistor_SMD:R_0402_1005Metric, F.Cu at (127.0, 58.3)
- added R6: 10k, Resistor_SMD:R_0402_1005Metric, F.Cu at (121.7, 58.0)
- added R7: 10k, Resistor_SMD:R_0402_1005Metric, F.Cu at (112.1, 66.9)
- added R8: 100k, Resistor_SMD:R_0402_1005Metric, F.Cu at (112.4, 60.6)
- added R9: 100k, Resistor_SMD:R_0402_1005Metric, F.Cu at (112.4, 61.6)
- added U3: MT2492, Package_TO_SOT_SMD:SOT-23-6, F.Cu at (124.3, 58.5)
- added U4: MT2492, Package_TO_SOT_SMD:SOT-23-6, F.Cu at (112.6, 64.3)
- added U5: MT2492, Package_TO_SOT_SMD:SOT-23-6, F.Cu at (112.6, 75.4)
- J1: value 2.54 -> Conn_02x12_Odd_Even; footprint Connector_PinHeader_2.54mm:PinHeader_1x12_P2.54mm_Vertical -> Connector_PinSocket_2.54mm:PinSocket_2x12_P2.54mm_Vertical
- SW1: value SW_SPST -> PTS645; footprint Button_Switch_SMD:SW_SPST_EVQQ2 -> Button_Switch_SMD:SW_SPST_PTS645
- moved SW1 12.8 mm to (151.5, 62.2), turned to 180 degrees
- moved C9 2.97 mm to (130.2, 88.0), turned to 180 degrees
- moved R3 2.83 mm to (147.4, 66.2), turned to 180 degrees
- moved R2 2.20 mm to (130.2, 89.0), turned to 180 degrees
- moved J1 1.77 mm to (119.0, 95.8)
- moved C10 1.57 mm to (124.8, 84.7), turned to 180 degrees
- moved C11 1.49 mm to (147.4, 67.2), turned to 0 degrees
- moved C5 0.60 mm to (124.8, 76.2)
- moved C7 0.30 mm to (130.2, 87.0)
- moved C4 0.16 mm to (141.8, 70.2)
Connections:
- C11 pad 1: Net-(U1D-RESET) -> Net-(SW1-A)
- J1 pad 1: /PE10 -> GND
- J1 pad 10: /UART_Tx -> /PE6
- J1 pad 11: /UART_Rx -> /PE11_CLKOUT
- J1 pad 12: GND -> /PE5
- J1 pad 2: /PE9 -> /PE10
- J1 pad 3: /PE8 -> /TWI0_SDA
- J1 pad 4: /PE7 -> /PE9
- J1 pad 5: /PE6 -> /UART1_Rx
- J1 pad 6: /PE5 -> /PE8
- J1 pad 7: /PE4 -> /UART1_Tx
- J1 pad 8: /PE3 -> /PE7
- J1 pad 9: /PE2 -> /TWI0_SCK
- J2 pad 1: VBUS -> +5V
- R3 pad 2: Net-(U1D-RESET) -> Net-(SW1-A)
- SW1 pad 1: unconnected-(SW1-A-Pad1) -> Net-(SW1-A)
- SW1 pad 2: unconnected-(SW1-B-Pad2) -> GND
- U1 pad 10: unconnected-(U1B-PD4-Pad10) -> /UART1_Tx
- U1 pad 70: Net-(U1D-RESET) -> Net-(SW1-A)
- U1 pad 9: unconnected-(U1B-PD3-Pad9) -> /UART1_Rx
Routing:
- net +3V3: track 16.6 -> 137.2 mm, vias 5 -> 13
- net +1V2: track 6.84 -> 70.2 mm, vias 3 -> 8
- net +2V5: track 11.3 -> 46.7 mm, vias 2 -> 7
- net Net-(SW1-A): track 0.00 -> 29.2 mm, vias 0 -> 2
- net /PD5: track 27.5 -> 0.00 mm
- net /PD6: track 25.7 -> 0.00 mm
- net /PD7: track 23.9 -> 0.00 mm
- net /PD8: track 22.2 -> 0.00 mm
- net /UART1_Rx: track 0.00 -> 21.4 mm, vias 0 -> 1
- net /UART1_Tx: track 0.00 -> 20.6 mm, vias 0 -> 1
- net /PD9: track 20.4 -> 0.00 mm
- net /PD10: track 18.6 -> 0.00 mm
- net /PD11: track 17.6 -> 0.00 mm
- net /PD13: track 15.8 -> 0.00 mm
- net /PE11_CLKOUT: track 25.3 -> 12.3 mm
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- added copper zone on F.Cu, net +1V2
- added copper zone on In2.Cu, net +1V2
- added copper zone on F.Cu, net +2V5
- added copper zone on In2.Cu, net +2V5
- added copper zone on F.Cu, net +3V3
- added copper zone on In2.Cu, net +3V3
- added copper zone on F.Cu, net +5V
- added copper zone on In2.Cu, net +5V
- added copper zone on F.Cu, net GND
- added copper zone on F.Cu, net Net-(U3-SW)
- added copper zone on F.Cu, net Net-(U4-SW)
- added copper zone on F.Cu, net Net-(U5-SW)
Other:
- copper layers 2 -> 4
