File: hardware/Orbital_imager_HiResDev_F1C200s/Orbital_imager_HiResDev_F1C200s.kicad_sch (KiCad schematic)
At the start: 26 parts, among them J1 2.54, J2 USB_B, J3 2.54, SW1 SW_SPST, U2 W25Q128, Y1 24MHz

Commit message: ported to C
Parts:
- removed J1, J3: 2.54, Connector_PinHeader_2.54mm:PinHeader_1x12_P2.54mm_Vertical, symbol Connector_Generic:Conn_01x12
- added C13: 1uF, Capacitor_SMD:C_0402_1005Metric, symbol Device:C_Small
- added C14, C19, C23: 22nF, Capacitor_SMD:C_0402_1005Metric, symbol Device:C_Small
- added C15, C16, C17, C18, C20, C21, C22, C24, C25: 22uF, Capacitor_SMD:C_0805_2012Metric, symbol Device:C_Small
- added D1: ESD0603, Diode_SMD:D_0603_1608Metric, symbol Diode:ESD5Zxx
- added D2: GREEN 0603, Diode_SMD:D_0603_1608Metric, symbol Device:LED
- added J1: Conn_02x12_Odd_Even, Connector_PinSocket_2.54mm:PinSocket_2x12_P2.54mm_Vertical, symbol Connector_Generic:Conn_02x12_Odd_Even
- added Le1, Le2, Le3: MPL2520S4R7MHT, Inductor_SMD:L_1008_2520Metric, symbol Device:L
- added R10, R13, R6, R7: 10k, Resistor_SMD:R_0402_1005Metric, symbol Device:R_Small
- added R11, R8, R9: 100k, Resistor_SMD:R_0402_1005Metric, symbol Device:R_Small
- added R12: 33k, Resistor_SMD:R_0402_1005Metric, symbol Device:R_Small
- added R4: 68k, Resistor_SMD:R_0402_1005Metric, symbol Device:R_Small
- added R5: 15k, Resistor_SMD:R_0402_1005Metric, symbol Device:R_Small
- added U3, U4, U5: MT2492, Package_TO_SOT_SMD:SOT-23-6, symbol Regulator_Switching:AP3211K
- SW1: value SW_SPST -> PTS645; footprint Button_Switch_SMD:SW_SPST_EVQQ2 -> Button_Switch_SMD:SW_SPST_PTS645
Connections:
- net +1V2: now also C20.1, C21.1, Le2.2, R8.1
- net +2V5: now also C24.1, C25.1, Le3.2, R11.1
- net +3V0: now also C13.1
- net +3V3: now also C15.1, C16.1, J1.21 (Pin_21), J1.23 (Pin_23), Le1.2, R4.1
- net GND: now also SW1.2 (B), C13.2, C15.2, C16.2, C17.2, C18.2, C20.2, C21.2, C22.2, C24.2, C25.2, D1.2 (A), J1.1 (Pin_1), J1.13 (Pin_13), J1.15 (Pin_15), J1.17 (Pin_17), J1.19 (Pin_19), J1.24 (Pin_24), R12.2, R13.2, R5.2, R9.2, U3.2 (GND), U4.2 (GND), U5.2 (GND)
- net PE10: now also J1.2 (Pin_2)
- net PE11_CLKOUT: now also J1.11 (Pin_11)
- net PE2: now also J1.18 (Pin_18)
- net PE3: now also J1.16 (Pin_16)
- net PE4: now also J1.14 (Pin_14)
- net PE5: now also J1.12 (Pin_12)
- net PE6: now also J1.10 (Pin_10)
- net PE7: now also J1.8 (Pin_8)
- net PE8: now also J1.6 (Pin_6)
- net PE9: now also J1.4 (Pin_4)
- net TWI0_SCK: now also J1.9 (Pin_9)
- net TWI0_SDA: now also J1.3 (Pin_3)
- net UART_Rx: now also J1.22 (Pin_22)
- net UART_Tx: now also J1.20 (Pin_20)
- net UART1_Tx: now reaches U1.10 (PD4)
- net UART1_Tx: now also J1.7 (Pin_7)
- net UART1_Rx: now reaches U1.9 (PD3)
- net UART1_Rx: now also J1.5 (Pin_5)
- net at SW1.1 (A): now also C11.1, R3.2, U1.70 (RESET)
- net VBUS renamed +5V
- net +5V: now also C17.1, C18.1, C22.1, D1.1 (K), D2.2 (A), R10.1, R6.1, R7.1, U3.5 (IN), U4.5 (IN), U5.5 (IN)
- new net: C19.2, U4.1 (BS)
- new net: R8.2, R9.1, U4.3 (FB)
- new net: R7.2, U4.4 (EN)
- new net: C19.1, Le2.1, U4.6 (SW)
- new net: R11.2, R12.1, U5.3 (FB)
- new net: C23.1, Le3.1, U5.6 (SW)
- new net: R10.2, U5.4 (EN)
- new net: R4.2, R5.1, U3.3 (FB)
- new net: R6.2, U3.4 (EN)
- new net: C23.2, U5.1 (BS)
- new net: D2.1 (K), R13.1
- new net: C14.1, Le1.1, U3.6 (SW)
- new net: C14.2, U3.1 (BS)
